File: USB2Speakon_PCB/USB2Speakon_PCB.kicad_sch (KiCad schematic)
At the start: 54 parts, among them J1 USB_C_Receptacle_USB2.0_16P, J2 Conn_01x04, U1 PCM2912A, U2 TPA2012D2RTJR, Y1 6 MHz

Commit message: replace crystal with oscillator and add solder pads for a capacitor
Parts:
- removed C3: 8p, Capacitor_SMD:C_0402_1005Metric, symbol Device:C_Small
- removed Y1: 6 MHz, Crystal:Crystal_SMD_3225-4Pin_3.2x2.5mm, symbol Device:Crystal_GND24_Small
- added C29: 100n, Capacitor_SMD:C_0402_1005Metric, symbol Device:C_Small
- added J3: Ext_Cap, Connector_PinSocket_2.54mm:PinSocket_1x02_P2.54mm_Vertical, symbol Connector_Generic:Conn_01x02
- added X1: 6MHz XO, LCSC:OSC-SMD_4P-L3.2-W2.5-BL, symbol Oscillator:XO32
- C2: value 8p -> DNP; now not fitted; now left out of the parts list
- J2: now left out of the parts list
- R4: value 1M -> DNP; now not fitted; now left out of the parts list
Connections:
- net GND: now also C29.1, J3.1 (Pin_1), X1.2 (GND); no longer C2.1
- net VBUS: now also JP1.1 (A), JP2.1 (A), R12.1, R9.1, U2.1 (G1), U2.15 (G0), J3.2 (Pin_2)
- net at R4.1: no longer U1.7 (XTO)
- net +3V3: now reaches C1.2, R3.2, U1.5 (VDD)
- net +3V3: now also C29.2, X1.4 (V+)
- new net: U1.8 (XTI), X1.3 (OUT)
- now unconnected: C2.2, R4.2
- no-connect marks 2 -> 7
Other:
- note added: "Dummy parts, so no new stencil is needed for v0.2"
